File: PrechargeV3/CANBUS.kicad_sch (KiCad schematic)
At the start: 5 parts, among them J3 436500228, U6 TCAN3404DRQ1

Commit message: Started Layout
Parts:
- C15: value K104K10X7RF5UH5 -> 1u; footprint 1uFCap:K104K10X7RF5UH5_VIS -> Capacitor_SMD:C_0805_2012Metric
- JP1: footprint Connector_PinHeader_1.00mm:PinHeader_1x02_P1.00mm_Vertical -> Connector_PinHeader_2.54mm:PinHeader_1x02_P2.54mm_Vertical
- R19: value R_US -> 120; footprint (none) -> Resistor_SMD:R_0603_1608Metric
Changed lines of the file:
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@@
 			)
 		)
-		(property "Value" "R_US"
+		(property "Value" "120"
 			(at 87.63 41.9099 0)
 			(effects
@@
 			)
 		)
-		(property "Footprint" ""
+		(property "Footprint" "Resistor_SMD:R_0603_1608Metric"
 			(at 86.106 40.894 90)
 			(effects
@@
 			)
 		)
-		(property "Footprint" "Connector_PinHeader_1.00mm:PinHeader_1x02_P1.00mm_Vertical"
+		(property "Footprint" "Connector_PinHeader_2.54mm:PinHeader_1x02_P2.54mm_Vertical"
 			(at 85.09 31.75 0)
 			(effects
@@
 			)
 		)
-		(property "Value" "K104K10X7RF5UH5"
+		(property "Value" "1u"
 			(at 50.8 34.2899 90)
 			(effects
@@
 			)
 		)
-		(property "Footprint" "1uFCap:K104K10X7RF5UH5_VIS"
+		(property "Footprint" "Capacitor_SMD:C_0805_2012Metric"
 			(at 46.99 29.21 0)
 			(effects
@@
 			)
 		)
-		(property "Datasheet" "K104K10X7RF5UH5"
+		(property "Datasheet" ""
 			(at 46.99 29.21 0)
 			(effects

Commit message: Finished Layout
Other:
- company: (none) -> Blake Hopper
- moved on the sheet: C15, J3, JP1, R19, U6

Commit message: Updated Layout
Parts:
- U6: footprint Package_TO_SOT_SMD:SOT-23-8 -> CAN interface:SOIC8_D_TEX
Changed lines of the file:
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@@
 			)
 		)
-		(property "Footprint" "Package_TO_SOT_SMD:SOT-23-8"
+		(property "Footprint" "CAN interface:SOIC8_D_TEX"
 			(at 64.77 43.18 0)
 			(effects
