File: PrechargeV3/PrechargeV3.kicad_pcb (KiCad board)
At the start: 2 copper layers, 84.5 x 50.2 mm, 66 parts, among them J1 430450428, J2 430450428, J3 436500228, J4 436500228, U1 NMV1S0505SC, U2 AMC1351DWVR, U3 AMC1351DWVR, U4 TLV9002QDGKRQ1, U7 MCP2551-I_SN, U8 MCP2515-I_SO, Y1 Crystal

Commit message: Started Layout
Parts:
- removed C13, C14: C, Capacitor_THT:C_Disc_D3.8mm_W2.6mm_P2.50mm
- removed CR1, CR2: B240A-13-F, RelayDriver:SMA_DIO
- removed MOSFET1, MOSFET2: DMN3404L-7, RelayDriver:SOT23_DIO
- removed U7: MCP2551-I_SN, CANBUS:SOIC127P599X175-8N
- removed U8: MCP2515-I_SO, CANBUS:SOIC127P1030X265-18N
- removed Y1: Crystal, Crystal:Crystal_HC49-U_Vertical
- added C16: 10u, Capacitor_SMD:C_1210_3225Metric, F.Cu at (119.2, 109.2)
- added C17: 10u, Capacitor_SMD:C_1210_3225Metric, F.Cu at (130.0, 77.2)
- added D1: B240A-13-F, Diodes:SMA_DIO, F.Cu at (180.9, 97.3)
- added D2: B240A-13-F, Diodes:SMA_DIO, F.Cu at (180.9, 82.0)
- added G***: LOGO, LOGO, F.Cu at (142.7, 66.8)
- added G***: LOGO, LOGO, F.Cu at (207.4, 81.5)
- added Q1: DMN3404L-7, MOSFETs:SOT23_DIO, F.Cu at (176.4, 101.6)
- added Q2: DMN3404L-7, MOSFETs:SOT23_DIO, F.Cu at (173.2, 85.2)
- added R19: 120, Resistor_SMD:R_0603_1608Metric, F.Cu at (175.4, 75.6)
- added R20: 0, Resistor_SMD:R_0805_2012Metric, F.Cu at (149.0, 88.3)
- added TP1: LV_in, TestPoint:TestPoint_Pad_D1.0mm, F.Cu at (134.2, 109.6)
- added TP10: INV_GND, TestPoint:TestPoint_Pad_D1.0mm, F.Cu at (117.0, 89.5)
- added TP11: BATT_GND, TestPoint:TestPoint_Pad_D1.0mm, F.Cu at (117.0, 99.2)
- added TP12: INV_+5, TestPoint:TestPoint_Pad_D1.0mm, F.Cu at (115.0, 77.0)
- added TP13: BATT_+5, TestPoint:TestPoint_Pad_D1.0mm, F.Cu at (115.0, 109.2)
- added TP2: GND, TestPoint:TestPoint_Pad_D1.0mm, F.Cu at (136.9, 74.4)
- added TP3: 5V, TestPoint:TestPoint_Pad_D1.0mm, F.Cu at (149.1, 102.0)
- added TP4: Vinv_LV+, TestPoint:TestPoint_Pad_D1.0mm, F.Cu at (133.0, 85.0)
- added TP5: Vinv_LV-, TestPoint:TestPoint_Pad_D1.0mm, F.Cu at (133.0, 87.1)
- added TP6: Vbatt_LV+, TestPoint:TestPoint_Pad_D1.0mm, F.Cu at (133.0, 94.4)
- added TP7: Vbatt_LV-, TestPoint:TestPoint_Pad_D1.0mm, F.Cu at (133.0, 96.9)
- added TP8: Inv_measured, TestPoint:TestPoint_Pad_D1.0mm, F.Cu at (147.9, 79.1)
- added TP9: Batt_Measured, TestPoint:TestPoint_Pad_D1.0mm, F.Cu at (146.3, 89.7)
- added U5: NMV1S0505SC, Isolating DC-DC Converters:SIP4_NMV1S0_MUR, F.Cu at (131.1, 105.8)
- added U6: TCAN3404DRQ1, Package_TO_SOT_SMD:SOT-23-8, F.Cu at (171.7, 72.0)
- C1, C11, C12: value C324C106K3R5TA -> 10u; footprint 10uF Cap:CAP_C324C_MR_X7R_KEM -> Capacitor_SMD:C_1210_3225Metric
- C10, C6, C7, C9: value K331K15X7RF5TL2 -> 330p; footprint 330pFCap:CAP_K-SERIES_15-L2_VIS -> Capacitor_SMD:C_0603_1608Metric
- C15, C2, C3, C4, C5, C8: value K104K10X7RF5UH5 -> 1u; footprint 1uFCap:K104K10X7RF5UH5_VIS -> Capacitor_SMD:C_0805_2012Metric
- J1, J2: footprint MolexVertical:CONN_SD-43045-010_04_MOL -> MolexConnectors:CONN_SD-43045-010_04_MOL
- J3, J4: footprint MolexVertical:CONN_SD-43650-010_02_MOL -> MolexConnectors:CONN_SD-43650-010_02_MOL
- JP1: footprint Connector_PinHeader_1.00mm:PinHeader_1x02_P1.00mm_Vertical -> Connector_PinHeader_2.54mm:PinHeader_1x02_P2.54mm_Vertical
- PS1: footprint 12-5V Converter:CONV_R-78E5.0-0.5 -> DC-DC Converters:R-78E5.0-0.5
- R1, R10, R11, R12, R13, R14, R15, R16, R17, R18, R2, R21, R22, R23, R24, R25, R26, R27, R28, R3, R4, R5, R6, R9: footprint Resistor_SMD:R_0603_1608Metric_Pad0.98x0.95mm_HandSolder -> Resistor_SMD:R_0603_1608Metric
- R7: value R_US -> 1.5k; footprint Resistor_SMD:R_0603_1608Metric_Pad0.98x0.95mm_HandSolder -> Resistor_SMD:R_0603_1608Metric
- R8: value R_US -> 1k; footprint Resistor_SMD:R_0603_1608Metric_Pad0.98x0.95mm_HandSolder -> Resistor_SMD:R_0603_1608Metric
- U1: value NMV1S0505SC -> AMC1351DWVR; footprint 5V-5V:SIP4_NMV1S0_MUR -> Isolating Amplifiers:SOIC8_DWV_TEX
- U2: footprint AMC 1351:SOIC8_DWV_TEX -> Isolating Amplifiers:SOIC8_DWV_TEX
- U3: value AMC1351DWVR -> TLV9002QDKRQ1; footprint AMC 1351:SOIC8_DWV_TEX -> OpAmps:VSSOP8_DGK_TEX
- U4: value TLV9002QDGKRQ1 -> NMV1S0505SC; footprint TLV9002:VSSOP8_DGK_TEX -> Isolating DC-DC Converters:SIP4_NMV1S0_MUR
- moved G*** 50.9 mm to (171.1, 60.5)
- moved G*** 50.5 mm to (157.4, 51.1)
- moved JP1 33.2 mm to (175.4, 69.1), turned to 0 degrees
- moved J3 29.2 mm to (182.0, 72.1), turned to 90 degrees
- moved C11 28.0 mm to (119.2, 77.2)
- moved C15 24.5 mm to (171.7, 68.3), turned to 180 degrees
- moved U3 20.1 mm to (143.2, 83.6), turned to -90 degrees
- moved U2 17.5 mm to (124.8, 96.2)
- moved R28 16.5 mm to (172.8, 88.1), turned to 0 degrees
- moved U1 16.0 mm to (124.8, 86.5), turned to 0 degrees
- moved U4 13.8 mm to (131.1, 73.8), turned to 180 degrees
- moved PS1 12.7 mm to (141.5, 98.9)
- moved R7 12.2 mm to (172.1, 93.4)
- moved R8 12.0 mm to (172.1, 96.6)
- moved R27 10.9 mm to (172.6, 82.2), turned to 0 degrees
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Connections:
- A1 pad A1: unconnected-(A1-PadA1) -> /InvMeasured
- A1 pad A2: Net-(U4-OUT2) -> unconnected-(A1-PadA2)
- A1 pad A4: unconnected-(A1-A4/SDA-PadA4) -> /BattMeasured
- A1 pad A7: Net-(U4-OUT1) -> unconnected-(A1-PadA7)
- A1 pad D10: nCS -> unconnected-(A1-PadD10)
- A1 pad D11: SI -> unconnected-(A1-D11_MOSI-PadD11)
- A1 pad D12: SO -> unconnected-(A1-D12_MISO-PadD12)
- A1 pad D13: SCK -> unconnected-(A1-D13_SCK-PadD13)
- A1 pad VIN: +5 -> +5V
- C1 pad 1: +5 -> +5V
- C10 pad 1: Net-(U4-IN2+) -> Net-(U3B-+)
- C11 pad 1: /HV+5 -> INV+5
- C11 pad 2: /HVGND -> INV_GND
- C12 pad 1: +5 -> +5V
- C15 pad 1: +5 -> GND
- C15 pad 2: GND -> +3.3V
- C2 pad 1: /HV+5 -> INV+5
- C2 pad 2: /HVGND -> INV_GND
- C3 pad 1: +5 -> +5V
- C4 pad 1: /HV+5 -> BATT+5
- C4 pad 2: /HVGND -> BATT_GND
- C5 pad 1: +5 -> +5V
- C6 pad 1: Net-(U4-IN1+) -> Net-(U3A-+)
- C7 pad 1: Net-(U4-IN1-) -> Net-(U3A--)
- C7 pad 2: Net-(U4-OUT1) -> /InvMeasured
- C8 pad 1: +5 -> +5V
- C9 pad 1: Net-(U4-IN2-) -> Net-(U3B--)
- C9 pad 2: Net-(U4-OUT2) -> /BattMeasured
- J2 pad 1: /HVGND -> Net-(J2-Pad1)
- J2 pad 2: /INVGND -> Net-(J2-Pad2)
- J2 pad 3: Net-(J2-Pad3) -> BATT_GND
- J2 pad 4: Net-(J2-Pad4) -> INV_GND
- J3 pad 2: Net-(JP1-B) -> Net-(U6-CANL)
- PS1 pad 3: +5 -> +5V
- R1 pad 1: Net-(J2-Pad4) -> Net-(J2-Pad2)
- R10 pad 1: Net-(U2-OUTP) -> Net-(U1-VOUTP)
- R10 pad 2: Net-(U4-IN1+) -> Net-(U3A-+)
- R11 pad 1: Net-(U4-OUT1) -> /InvMeasured
- R11 pad 2: Net-(U4-IN1-) -> Net-(U3A--)
- R12 pad 2: Net-(U4-IN1+) -> Net-(U3A-+)
- R13 pad 1: Net-(J2-Pad3) -> Net-(J2-Pad1)
- R17 pad 2: Net-(U3-IN) -> Net-(U2-VINP)
- R18 pad 1: /HVGND -> BATT_GND
- R18 pad 2: Net-(U3-IN) -> Net-(U2-VINP)
- R21 pad 1: Net-(U3-OUTP) -> Net-(U2-VOUTP)
- R21 pad 2: Net-(U4-IN2+) -> Net-(U3B-+)
- R22 pad 1: Net-(U3-OUTN) -> Net-(U2-VOUTN)
- R22 pad 2: Net-(U4-IN2-) -> Net-(U3B--)
- R23 pad 2: Net-(U4-IN2+) -> Net-(U3B-+)
- R24 pad 1: Net-(U4-OUT2) -> /BattMeasured
- R24 pad 2: Net-(U4-IN2-) -> Net-(U3B--)
- R5 pad 2: Net-(U2-IN) -> Net-(U1-VINP)
- R6 pad 1: /INVGND -> INV_GND
- R6 pad 2: Net-(U2-IN) -> Net-(U1-VINP)
- R9 pad 1: Net-(U2-OUTN) -> Net-(U1-VOUTN)
- R9 pad 2: Net-(U4-IN1-) -> Net-(U3A--)
- U1 pad 1: +5 -> INV+5
- U1 pad 2: GND -> Net-(U1-VINP)
- U1 pad 5: /HVGND -> GND
- U1 pad 7: /HV+5 -> Net-(U1-VOUTP)
- U2 pad 1: /HV+5 -> BATT+5
- U2 pad 2: Net-(U2-IN) -> Net-(U2-VINP)
- U2 pad 3: /INVGND -> BATT_GND
- U2 pad 4: /INVGND -> BATT_GND
- U2 pad 6: Net-(U2-OUTN) -> Net-(U2-VOUTN)
- U2 pad 7: Net-(U2-OUTP) -> Net-(U2-VOUTP)
- U2 pad 8: +5 -> +5V
- U3 pad 1: /HV+5 -> /InvMeasured
- U3 pad 2: Net-(U3-IN) -> Net-(U3A--)
- U3 pad 3: /HVGND -> Net-(U3A-+)
- U3 pad 4: /HVGND -> GND
- U3 pad 5: GND -> Net-(U3B-+)
- U3 pad 6: Net-(U3-OUTN) -> Net-(U3B--)
- U3 pad 7: Net-(U3-OUTP) -> /BattMeasured
- U3 pad 8: +5 -> +5V
- U4 pad 1: Net-(U4-OUT1) -> +5V
- U4 pad 2: Net-(U4-IN1-) -> GND
- U4 pad 5: Net-(U4-IN2+) -> INV_GND
- U4 pad 7: Net-(U4-OUT2) -> INV+5
Routing:
- net +5: track 116.3 -> 0.00 mm, vias 1 -> 0
- net +5V: track 0.00 -> 97.1 mm
- net BATT_GND: track 0.00 -> 46.1 mm, vias 0 -> 1
- net Net-(U4-OUT2): track 40.1 -> 0.00 mm, vias 1 -> 0
- net /HV+5: track 39.5 -> 0.00 mm
- net Net-(U4-OUT1): track 38.5 -> 0.00 mm, vias 1 -> 0
- net INV_GND: track 0.00 -> 36.0 mm, vias 0 -> 1
- net nCS: track 29.2 -> 0.00 mm
- net SO: track 27.5 -> 0.00 mm, vias 1 -> 0
- net SI: track 27.0 -> 0.00 mm
- net CANInt: track 25.5 -> 0.00 mm, vias 1 -> 0
- net /ShutdownIn: track 25.3 -> 0.00 mm
- net BATT+5: track 0.00 -> 22.6 mm, vias 0 -> 1
- net Net-(U4-IN2-): track 17.2 -> 0.00 mm
- net Net-(JP1-A): track 16.2 -> 0.00 mm
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- added copper zone on B.Cu, net BATT_GND
- added copper zone on B.Cu, net INV_GND
- removed copper zone on B.Cu, net /HVGND
- removed copper zone on F.Cu, net /HVGND
Other:
- board size 84.5 x 50.2 mm -> 79.2 x 52.8 mm
- board text added: "Precharge V3"
- board text removed: "Precharge V2"

Commit message: Finished Layout
Parts:
- removed the G*** at (157.4, 51.1)
- removed the G*** at (207.4, 81.5)
- A1: footprint PCM_arduino-library:Arduino_Nano_33_IoT_Socket -> MCUs:Arduino_Nano_33_IoT_Socket
- moved C15 6.75 mm to (172.8, 75.0)
- moved R8 5.90 mm to (173.7, 90.9)
- moved R25 3.37 mm to (172.8, 97.2)
- moved Q1 3.33 mm to (173.2, 100.4)
- moved R7 2.84 mm to (170.6, 91.0)
- moved J4 1.98 mm to (140.8, 108.5)
- moved G*** 1.75 mm to (142.8, 68.6)
- moved R27 1.40 mm to (172.6, 80.8)
- moved R26 1.33 mm to (172.8, 103.6)
- moved D1 1.16 mm to (179.8, 97.5)
- moved JP1 1.14 mm to (176.3, 68.4)
- moved R19 1.14 mm to (176.3, 75.0)
- moved Q2 1.14 mm to (173.1, 84.0)
- moved D2 1.03 mm to (179.9, 81.8)
- moved REF** 1.00 mm to (181.2, 107.7)
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Connections:
- A1 pad D10: unconnected-(A1-PadD10) -> RX
- A1 pad D2: Net-(A1-PadD2) -> TX
- A1 pad D3: /PrechargeStatus -> Net-(A1-PadD3)
- A1 pad D4: /SenseSHD -> /PrechargeStatus
- A1 pad D5: unconnected-(A1-PadD5) -> /SenseSHD
- A1 pad D8: CANInt -> unconnected-(A1-PadD8)
- R25 pad 1: Net-(A1-PadD2) -> Net-(A1-PadD3)
Routing:
- net TX: track 0.00 -> 28.2 mm, vias 0 -> 1
- net /ShutdownIn: track 0.00 -> 27.2 mm
- net Net-(Q2-D): track 0.00 -> 24.6 mm
- net Net-(Q1-D): track 0.00 -> 20.9 mm
- net GND: track 15.2 -> 36.1 mm, vias 5 -> 23
- net /PrechargeStatus: track 0.00 -> 13.2 mm, vias 0 -> 1
- net Net-(JP1-A): track 0.00 -> 12.0 mm
- net Net-(U6-CANL): track 0.00 -> 11.3 mm
- net Net-(Q2-G): track 0.00 -> 8.93 mm
- net Net-(Q1-G): track 0.00 -> 8.74 mm
- net /SenseSHD: track 0.00 -> 8.49 mm
- net Net-(A1-PadD3): track 0.00 -> 5.88 mm
- net Net-(A1-PadD9): track 0.00 -> 5.23 mm
- net RX: track 0.00 -> 4.67 mm
- net +3.3V: track 0.00 -> 3.73 mm
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
Commit message: Updated Layout
Parts:
- R1, R13, R14, R15, R16, R17, R18, R2, R3, R4, R5, R6: footprint Resistor_SMD:R_0603_1608Metric -> Capacitor_SMD:C_0805_2012Metric
- U6: footprint Package_TO_SOT_SMD:SOT-23-8 -> CAN interface:SOIC8_D_TEX
- moved Q2 5.98 mm to (178.4, 81.4)
- moved Q1 5.92 mm to (178.3, 103.6)
- moved R7 5.24 mm to (175.8, 90.0), turned to 0 degrees
- moved D1 4.46 mm to (183.1, 100.3)
- moved D2 4.46 mm to (183.3, 84.7)
- moved J1 4.46 mm to (185.3, 91.1)
- moved R28 4.38 mm to (172.9, 82.9), turned to -90 degrees
- moved R25 3.68 mm to (174.9, 100.2)
- moved G*** 3.42 mm to (174.5, 60.5)
- moved JP1 3.42 mm to (179.8, 68.5)
- moved R19 3.42 mm to (179.8, 75.0)
- moved REF** 3.42 mm to (184.6, 107.7)
- moved REF** 3.42 mm to (184.6, 62.0)
- moved J3 3.42 mm to (185.4, 72.1)
- moved C15 2.39 mm to (174.6, 76.6)
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Connections:
- A1 pad 5V: unconnected-(A1-Pad5V) -> +5V
Routing:
- net TX: track 28.2 -> 40.2 mm, vias 1 -> 0
- net Net-(Q2-D): track 24.6 -> 18.5 mm
- net GND: track 36.1 -> 41.6 mm, vias 23 -> 17
- net +5V: track 94.9 -> 99.8 mm
- net INV+5: track 12.8 -> 17.5 mm
- net Net-(A1-PadD3): track 5.88 -> 9.47 mm
- net Net-(Q2-G): track 8.93 -> 5.62 mm
- net Net-(Q1-D): track 20.9 -> 17.7 mm
- net /PrechargeStatus: track 13.2 -> 16.0 mm
- net Net-(Q1-G): track 8.74 -> 5.96 mm
- net BATT+5: track 22.6 -> 25.3 mm
- net INV_GND: track 36.0 -> 33.2 mm
- net Net-(U3A--): track 4.42 -> 7.13 mm
- net /ShutdownIn: track 27.2 -> 25.0 mm
- net Net-(U3B--): track 5.14 -> 7.06 mm
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Other:
- board size 79.2 x 52.8 mm -> 82.4 x 52.8 mm

Commit message: Precharge state machine & 3.3v component adjustments
Precharge state machine written for stm32. Differential op-amp and shutdown sense resistor values changed from 5v logic level mcu to 3.3v one.
Parts:
- R10, R21, R22, R9: value 1k -> 9.09k
- R11, R12, R23, R24: value 2.5k -> 15k
- R7: value 1.5k -> 3.01k
Changed lines of the file:
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@@
 			)
 		)
-		(property "Value" "2.5k"
+		(property "Value" "15k"
 			(at 0 1.43 180)
 			(layer "F.Fab")
@@
 			)
 		)
-		(property "Value" "1k"
+		(property "Value" "9.09k"
 			(at 0 1.43 0)
 			(layer "F.Fab")
@@
 			)
 		)
-		(property "Value" "2.5k"
+		(property "Value" "15k"
 			(at 0 1.43 0)
 			(layer "F.Fab")
@@
 			)
 		)
-		(property "Value" "1k"
+		(property "Value" "9.09k"
 			(at 0 1.43 0)
 			(layer "F.Fab")
@@
 			)
 		)
-		(property "Value" "2.5k"
+		(property "Value" "15k"
 			(at 0 1.43 0)
 			(layer "F.Fab")
@@
 			)
 		)
-		(property "Value" "1.5k"
+		(property "Value" "3.01k"
 			(at 0 1.43 0)
 			(layer "F.Fab")
@@
 			)
 		)
-		(property "Value" "2.5k"
+		(property "Value" "15k"
 			(at 0 1.43 180)
 			(layer "F.Fab")
@@
 			)
 		)
-		(property "Value" "1k"
+		(property "Value" "9.09k"
 			(at 0 1.43 0)
 			(layer "F.Fab")
@@
 			)
 		)
-		(property "Value" "1k"
+		(property "Value" "9.09k"
 			(at 0 1.43 0)
 			(layer "F.Fab")
